File: subsheet_03.kicad_sch (KiCad schematic)
At the start: 1 part, among them U2 GATE_ARRAY_MO5_V2_SOCKET

Commit message: done schematics
Parts:
- renumbered U2 to U4
Connections:
- net GND: now reaches U4.1 (GND)
- net GND: now also U4.17 (GND), U4.35 (GND)
- net +5V: now reaches U4.18 (VCC)
- net +5V: now also U4.2 (VCC), U4.52 (VCC)
- net E: now reaches U4.41 (E)
- net 16MHz: now reaches U4.46 (H16)
- no-connect marks 0 -> 60
